Commit message: Initial commit

File: morus_description/urdf/morus.gazebo.xacro (robot description, xacro)
@@ -122,6 +122,3 @@
     <origin xyz="-0.0 0.0 0" rpy="0.0 0.0 0.0" />
   </xacro:odometry_plugin_macro>
-  <gazebo reference="base_link">
-    <dampingFactor>0.0003</dampingFactor>
-  </gazebo>
 </robot>

File: morus_description/urdf/morus.urdf.xacro (robot description, xacro)
@@ -3,26 +3,24 @@
   <!-- Properties -->
   <xacro:property name="rotor_velocity_slowdown_sim" value="10" />
-  <xacro:arg name="custom_mesh_file" default="morus_uav_final.dae" />
-  <xacro:property name="mesh_file" value="$(arg custom_mesh_file)" />
+  <xacro:property name="mesh_file" value="MORUS_UAV_without_mass.dae" />
   <xacro:property name="mesh_file_mass" value="MORUS_mass.dae" />
   <xacro:property name="mass" value="30" />  <!-- [kg] -->
-   <xacro:property name="body_width" value="0.35" /> <!-- 0.1 [m] -->
-  <xacro:property name="body_height" value="0.15" /> <!--0.2 [m] -->
+  <xacro:property name="body_width" value="0.3" /> <!-- 0.1 [m] -->
+  <xacro:property name="body_height" value="0.25" /> <!--0.2 [m] -->
   <xacro:property name="mass_rotor" value="0.2" /> <!-- [kg] -->
-  <xacro:property name="arm_length" value="0.65" /> <!-- [m] -->
-  <xacro:property name="arm_offset" value="0.175" /> <!-- [m] -->
-  <xacro:property name="prop_ver_offset" value="0.15" /> <!-- [m] -->
-  <xacro:property name="prop_long_offset" value="0.07" /> <!-- [m] -->
+  <xacro:property name="arm_length" value="0.515" /> <!-- [m] -->
+  <xacro:property name="arm_offset" value="0.1" /> <!-- [m] -->
+  <xacro:property name="propeler_offset" value="0.325" /> <!-- [m] -->
+  <xacro:property name="rotor_offset_top" value="0.037" /> <!-- [m] -->
   <xacro:property name="radius_rotor" value="0.33" /> <!-- [m] -->
   <xacro:property name="motor_constant" value="0.000456874" /> <!-- [kg*m/s^2] -->
-  <xacro:property name="moment_constant" value="0.025" /> <!-- [m] -->
-  <xacro:property name="time_constant_up" value="0.2" /> <!-- [s] -->
-  <xacro:property name="time_constant_down" value="0.2" /> <!-- [s] -->
+  <xacro:property name="moment_constant" value="0.01" /> <!-- [m] -->
+  <xacro:property name="time_constant" value="0.125" /> <!-- [s] -->s ti
   <xacro:property name="max_rot_velocity" value="838" /> <!-- [rad/s] -->
-  <xacro:property name="rotor_drag_coefficient" value="0.0" /> <!--8.06428e-03-->
+  <xacro:property name="rotor_drag_coefficient" value="8.06428e-04" />
   <xacro:property name="rolling_moment_coefficient" value="0.00001" />
   <xacro:property name="movable_mass_mass" value="1" />
   <xacro:property name="movable_mass_dimension" value="0.08" />
-  <xacro:property name="movable_mass_offset" value="0.05" />
+  <xacro:property name="movable_mass_offset" value="0.025" />
   <xacro:property name="imu_mass" value="0.02"/>
   <xacro:property name="imu_size" value="0.01"/>
@@ -32,6 +30,5 @@
   <!-- Property Blocks -->
   <xacro:property name="body_inertia">
-    <!--inertia ixx="8.66" ixy="0.0" ixz="0.0" iyy="8.66" iyz="0.0" izz="12.0" /!-->
-    <inertia ixx="5.5" ixy="0.0" ixz="0.0" iyy="5.5" iyz="0.0" izz="6.5" />
+    <inertia ixx="5.5268" ixy="0.0" ixz="0.0" iyy="5.5268" iyz="0.0" izz="6.8854" />
   </xacro:property>
   <!-- inertia of a single rotor, assuming it is a cuboid. Height=3mm, width=15mm -->
@@ -71,5 +68,5 @@
     <xacro:insert_block name="body_inertia" />
   </xacro:multirotor_base_macro>
- <!-- Instantiate rotors -->
+  <!-- Instantiate rotors -->
   <xacro:vertical_rotor
     robot_namespace="$(arg name)"
@@ -81,6 +78,5 @@
     mass_rotor="${mass_rotor}"
     radius_rotor="${radius_rotor}"
-    time_constant_up="${time_constant_up}"
-    time_constant_down="${time_constant_down}"
+    time_constant="${time_constant}"
     max_rot_velocity="${max_rot_velocity}"
     motor_number="0"
@@ -88,5 +84,5 @@
     rolling_moment_coefficient="${rolling_moment_coefficient}"
     color="Red">
-    <origin xyz="${arm_length+prop_long_offset+arm_offset} 0 ${prop_ver_offset}" rpy="0 0 0" />
+    <origin xyz="${arm_length+arm_offset} 0 ${propeler_offset}" rpy="0 0 0" />
     <xacro:insert_block name="rotor_inertia" />
   </xacro:vertical_rotor>
@@ -100,6 +96,5 @@
     mass_rotor="${mass_rotor}"
     radius_rotor="${radius_rotor}"
-    time_constant_up="${time_constant_up}"
-    time_constant_down="${time_constant_down}"
+    time_constant="${time_constant}"
     max_rot_velocity="${max_rot_velocity}"
     motor_number="1"
@@ -107,5 +102,5 @@
     rolling_moment_coefficient="${rolling_moment_coefficient}"
     color="Blue">
-    <origin xyz="0 ${arm_length+prop_long_offset+arm_offset} ${prop_ver_offset}" rpy="0 0 0" />
+    <origin xyz="0 ${arm_length+arm_offset} ${propeler_offset}" rpy="0 0 0" />
     <xacro:insert_block name="rotor_inertia" />
   </xacro:vertical_rotor>
@@ -119,6 +114,5 @@
     mass_rotor="${mass_rotor}"
     radius_rotor="${radius_rotor}"
-    time_constant_up="${time_constant_up}"
-    time_constant_down="${time_constant_down}"
+    time_constant="${time_constant}"
     max_rot_velocity="${max_rot_velocity}"
     motor_number="2"
@@ -126,5 +120,5 @@
     rolling_moment_coefficient="${rolling_moment_coefficient}"
     color="Blue">
-    <origin xyz="${-(arm_length+prop_long_offset+arm_offset)} 0 ${prop_ver_offset}" rpy="0 0 0" />
+    <origin xyz="${-(arm_length+arm_offset)} 0 ${propeler_offset}" rpy="0 0 0" />
     <xacro:insert_block name="rotor_inertia" />
   </xacro:vertical_rotor>
@@ -138,6 +132,5 @@
     mass_rotor="${mass_rotor}"
     radius_rotor="${radius_rotor}"
-    time_constant_up="${time_constant_up}"
-    time_constant_down="${time_constant_down}"
+    time_constant="${time_constant}"
     max_rot_velocity="${max_rot_velocity}"
     motor_number="3"
@@ -145,5 +138,5 @@
     rolling_moment_coefficient="${rolling_moment_coefficient}"
     color="Blue">
-    <origin xyz="0 ${-(arm_length+prop_long_offset+arm_offset)} ${prop_ver_offset}" rpy="0 0 0" />
+    <origin xyz="0 ${-(arm_length+arm_offset)} ${propeler_offset}" rpy="0 0 0" />
     <xacro:insert_block name="rotor_inertia" />
   </xacro:vertical_rotor>
@@ -186,5 +179,5 @@
     y_axis="0"
     z_axis="0"
-    orientation="${PI}">
+    orientation="${PI}">>
     <origin xyz="${-(arm_length/2+arm_offset)} 0.0 ${movable_mass_offset}" rpy="0 0 0" />
     <xacro:insert_block name="movable_mass_inertia"/>
@@ -200,5 +193,5 @@
     y_axis="-1"
     z_axis="0"
-    orientation="${PI/2}">
+    orientation="${PI/2}">>
     <origin xyz="0.0 ${-(arm_length/2+arm_offset)} ${movable_mass_offset}" rpy="0 0 0" />
     <xacro:insert_block name="movable_mass_inertia"/>
@@ -231,8 +224,8 @@
       gear_num = "1"
       mass = "1e-6"
-      dim_x = "0.12"
-      dim_y = "0.04"
-      dim_z = "0.0001">
-      <origin xyz="0 -0.7 -0.275" rpy="0 0 0" />
+      dim_x = "0.8"
+      dim_y = "0.1"
+      dim_z = "0.05">
+      <origin xyz="0 -0.325 -0.6" rpy="0 0 0" />
       <xacro:insert_block name="land_gear_inertia"/>
   </xacro:landing_gear>
@@ -241,28 +234,8 @@
       gear_num = "2"
       mass = "1e-6"
-      dim_x = "0.12"
-      dim_y = "0.04"
-      dim_z = "0.0001">
-      <origin xyz="0 0.7 -0.275" rpy="0 0 0" />
-      <xacro:insert_block name="land_gear_inertia"/>
-  </xacro:landing_gear>
-  <xacro:landing_gear
-      parent="base_link"
-      gear_num = "3"
-      mass = "1e-6"
-      dim_x = "0.12"
-      dim_y = "0.04"
-      dim_z = "0.0001">
-      <origin xyz="-0.7 0 -0.275" rpy="0 0 1.57" />
-      <xacro:insert_block name="land_gear_inertia"/>
-  </xacro:landing_gear>
-  <xacro:landing_gear
-      parent="base_link"
-      gear_num = "4"
-      mass = "1e-6"
-      dim_x = "0.12"
-      dim_y = "0.04"
-      dim_z = "0.0001">
-      <origin xyz="0.7 0.0 -0.275" rpy="0 0 1.57" />
+      dim_x = "0.8"
+      dim_y = "0.1"
+      dim_z = "0.05">
+      <origin xyz="0 0.325 -0.6" rpy="0 0 0" />
       <xacro:insert_block name="land_gear_inertia"/>
   </xacro:landing_gear>

File: morus_description/urdf/multirotor_base.urdf.xacro (robot description, xacro)
@@ -17,8 +17,8 @@
       </inertial>
       <visual>
-        <origin xyz="0 0 -0.65" rpy="0 0 0" />
+        <origin xyz="0 0 0.125" rpy="0 0 0" />
         <geometry>
           <mesh filename="package://morus_description/meshes/${mesh_file}"
-            scale="0.001 0.001 0.001" />
+            scale="1 1 1" />
           <!--box size="${body_width} ${body_width} ${body_height}"/--> <!-- [m] [m] [m] -->
         </geometry>
@@ -71,5 +71,5 @@
       <visual>
         <!--origin rpy="0 0 ${orientation}" xyz="0 0 ${0*movable_mass_dimension/2}"/-->
-        <origin rpy="0 0 ${orientation}" xyz="0 0 -0.05"/>
+        <origin rpy="0 0 ${orientation}" xyz="0 0 0"/>
         <geometry>
           <!--mesh filename="package://morus_description/meshes/${mesh_file_mass}"
@@ -96,5 +96,5 @@
   <!-- Rotor joint and link -->
   <xacro:macro name="vertical_rotor"
-    params="robot_namespace suffix direction motor_constant moment_constant parent mass_rotor radius_rotor time_constant_up time_constant_down max_rot_velocity motor_number rotor_drag_coefficient rolling_moment_coefficient color *origin *inertia">
+    params="robot_namespace suffix direction motor_constant moment_constant parent mass_rotor radius_rotor time_constant max_rot_velocity motor_number rotor_drag_coefficient rolling_moment_coefficient color *origin *inertia">
     <joint name="rotor_${motor_number}_joint" type="continuous">
       <xacro:insert_block name="origin" />
@@ -132,6 +132,5 @@
         <linkName>rotor_${motor_number}</linkName>
         <turningDirection>${direction}</turningDirection>
-        <timeConstantUp>${time_constant_up}</timeConstantUp>
-        <timeConstantDown>${time_constant_down}</timeConstantDown>
+        <timeConstant>${time_constant}</timeConstant>
         <maxRotVelocity>${max_rot_velocity}</maxRotVelocity>
         <motorConstant>${motor_constant}</motorConstant>
