Commit message: Added launch files

File: morus_description/urdf/morus.base.urdf.xacro (robot description, xacro)
@@ -58,4 +58,77 @@
   <!-- Included URDF Files -->
   <xacro:include filename="$(find morus_description)/urdf/multirotor_base.urdf.xacro" />
+  <!-- Instantiate rotors -->
+  <xacro:vertical_rotor
+    robot_namespace="$(arg name)"
+    suffix="front"
+    direction="cw"
+    motor_constant="${motor_constant}"
+    moment_constant="${moment_constant}"
+    parent="base_link"
+    mass_rotor="${mass_rotor}"
+    radius_rotor="${radius_rotor}"
+    time_constant="${time_constant}"
+    max_rot_velocity="${max_rot_velocity}"
+    motor_number="0"
+    rotor_drag_coefficient="${rotor_drag_coefficient}"
+    rolling_moment_coefficient="${rolling_moment_coefficient}"
+    color="Red">
+    <origin xyz="${arm_length+arm_offset} 0 ${propeler_offset}" rpy="0 0 0" />
+    <xacro:insert_block name="rotor_inertia" />
+  </xacro:vertical_rotor>
+  <xacro:vertical_rotor
+    robot_namespace="$(arg name)"
+    suffix="left"
+    direction="ccw"
+    motor_constant="${motor_constant}"
+    moment_constant="${moment_constant}"
+    parent="base_link"
+    mass_rotor="${mass_rotor}"
+    radius_rotor="${radius_rotor}"
+    time_constant="${time_constant}"
+    max_rot_velocity="${max_rot_velocity}"
+    motor_number="1"
+    rotor_drag_coefficient="${rotor_drag_coefficient}"
+    rolling_moment_coefficient="${rolling_moment_coefficient}"
+    color="Blue">
+    <origin xyz="0 ${arm_length+arm_offset} ${propeler_offset}" rpy="0 0 0" />
+    <xacro:insert_block name="rotor_inertia" />
+  </xacro:vertical_rotor>
+  <xacro:vertical_rotor
+    robot_namespace="$(arg name)"
+    suffix="back"
+    direction="cw"
+    motor_constant="${motor_constant}"
+    moment_constant="${moment_constant}"
+    parent="base_link"
+    mass_rotor="${mass_rotor}"
+    radius_rotor="${radius_rotor}"
+    time_constant="${time_constant}"
+    max_rot_velocity="${max_rot_velocity}"
+    motor_number="2"
+    rotor_drag_coefficient="${rotor_drag_coefficient}"
+    rolling_moment_coefficient="${rolling_moment_coefficient}"
+    color="Blue">
+    <origin xyz="${-(arm_length+arm_offset)} 0 ${propeler_offset}" rpy="0 0 0" />
+    <xacro:insert_block name="rotor_inertia" />
+  </xacro:vertical_rotor>
+  <xacro:vertical_rotor
+    robot_namespace="$(arg name)"
+    suffix="right"
+    direction="ccw"
+    motor_constant="${motor_constant}"
+    moment_constant="${moment_constant}"
+    parent="base_link"
+    mass_rotor="${mass_rotor}"
+    radius_rotor="${radius_rotor}"
+    time_constant="${time_constant}"
+    max_rot_velocity="${max_rot_velocity}"
+    motor_number="3"
+    rotor_drag_coefficient="${rotor_drag_coefficient}"
+    rolling_moment_coefficient="${rolling_moment_coefficient}"
+    color="Blue">
+    <origin xyz="0 ${-(arm_length+arm_offset)} ${propeler_offset}" rpy="0 0 0" />
+    <xacro:insert_block name="rotor_inertia" />
+  </xacro:vertical_rotor>
   <!-- Instantiate multirotor_base_macro once-->
   <xacro:multirotor_base_macro

File: morus_description/urdf/morus.gazebo.xacro (robot description, xacro)
@@ -100,4 +100,5 @@
     pose_topic="pose"
     pose_with_covariance_topic="pose_with_covariance"
+    velocity_relative_topic="velocity_relative"
     position_topic="position"
     transform_topic="transform"

File: morus_description/urdf/morus.urdf.xacro (robot description, xacro)
@@ -142,5 +142,5 @@
   </xacro:vertical_rotor>
   <!-- Instantiate movable mass 0-->
-  <xacro:movable_mass
+  <!--xacro:movable_mass
     mass_number="0"
     parent="base_link"
@@ -154,7 +154,7 @@
     <origin xyz="${(arm_length/2+arm_offset)} 0.0 ${movable_mass_offset}" rpy="0 0 0" />
     <xacro:insert_block name="movable_mass_inertia"/>
-  </xacro:movable_mass>
+  </xacro:movable_mass-->
   <!-- Instantiate movable mass 1 -->
-  <xacro:movable_mass
+  <!--xacro:movable_mass
     mass_number="1"
     parent="base_link"
@@ -168,7 +168,7 @@
     <origin xyz="0.0 ${(arm_length/2+arm_offset)} ${movable_mass_offset}" rpy="0 0 0" />
     <xacro:insert_block name="movable_mass_inertia"/>
-  </xacro:movable_mass>
+  </xacro:movable_mass-->
   <!-- Instantiate movable mass 2-->
-  <xacro:movable_mass
+  <!--xacro:movable_mass
     mass_number="2"
     parent="base_link"
@@ -182,7 +182,7 @@
     <origin xyz="${-(arm_length/2+arm_offset)} 0.0 ${movable_mass_offset}" rpy="0 0 0" />
     <xacro:insert_block name="movable_mass_inertia"/>
-  </xacro:movable_mass>
+  </xacro:movable_mass-->
   <!-- Instantiate movable mass 3 -->
-  <xacro:movable_mass
+  <!--xacro:movable_mass
     mass_number="3"
     parent="base_link"
@@ -196,5 +196,6 @@
     <origin xyz="0.0 ${-(arm_length/2+arm_offset)} ${movable_mass_offset}" rpy="0 0 0" />
     <xacro:insert_block name="movable_mass_inertia"/>
-  </xacro:movable_mass>
+  </xacro:movable_mass-->
+<!--
   <xacro:transmisija
     trans_number="0"
@@ -213,4 +214,5 @@
     joint_name="stick_to_movable_mass_3">
   </xacro:transmisija>
+-->
   <xacro:property name="land_gear_inertia">
     <inertia
