Commit message: Removed multirotor body mesh

File: morus_description/urdf/multirotor_base.urdf.xacro (robot description, xacro)
@@ -19,7 +19,7 @@
         <origin xyz="0 0 0.125" rpy="0 0 0" />
         <geometry>
-          <mesh filename="package://morus_description/meshes/${mesh_file}"
-            scale="1 1 1" />
-          <!--box size="${body_width} ${body_width} ${body_height}"/--> <!-- [m] [m] [m] -->
+          <!--mesh filename="package://morus_description/meshes/${mesh_file}"
+            scale="1 1 1" /-->
+          <box size="${body_width} ${body_width} ${body_height}"/> <!-- [m] [m] [m] -->
         </geometry>
       </visual>

Commit message: started yaw implementation

File: morus_description/urdf/multirotor_base.urdf.xacro (robot description, xacro)
@@ -19,7 +19,7 @@
         <origin xyz="0 0 0.125" rpy="0 0 0" />
         <geometry>
-          <!--mesh filename="package://morus_description/meshes/${mesh_file}"
-            scale="1 1 1" /-->
-          <box size="${body_width} ${body_width} ${body_height}"/> <!-- [m] [m] [m] -->
+          <mesh filename="package://morus_description/meshes/${mesh_file}"
+            scale="1 1 1" />
+          <!--box size="${body_width} ${body_width} ${body_height}"/--> <!-- [m] [m] [m] -->
         </geometry>
       </visual>

Commit message: Drone days 2019, Initial commit

File: morus_description/urdf/multirotor_base.urdf.xacro (robot description, xacro)
@@ -73,7 +73,7 @@
         <origin rpy="0 0 ${orientation}" xyz="0 0 0"/>
         <geometry>
-          <!--mesh filename="package://morus_description/meshes/${mesh_file_mass}"
-            scale="1 1 1" /-->
-          <box size="${1*dimension} ${1*dimension} ${1*dimension}"/>
+          <mesh filename="package://morus_description/meshes/${mesh_file_mass}"
+            scale="1 1 1" />
+          <!-- box size="${1*dimension} ${1*dimension} ${1*dimension}"/ -->
         </geometry>
       </visual>
