Commit message: initial commit

File: morus_description/urdf/morus.urdf.xacro (robot description, xacro)
@@ -68,4 +68,56 @@
     <xacro:insert_block name="body_inertia" />
   </xacro:multirotor_base_macro>
+  <!-- Instantiate tilt 0-->
+  <xacro:tilt
+    motor_number="0"
+    parent="base_link"
+    color="Red"
+    x_axis="1"
+    y_axis="0">
+    <origin xyz="${arm_length+arm_offset} 0 0" rpy="0 0 0" />
+  </xacro:tilt>
+  <!-- Instantiate tilt 1 -->
+  <xacro:tilt
+    motor_number="1"
+    parent="base_link"
+    color="Blue"
+    x_axis="0"
+    y_axis="1">
+    <origin xyz="0 ${arm_length+arm_offset} 0" rpy="0 0 0" />
+  </xacro:tilt>
+  <!-- Instantiate tilt 2-->
+  <xacro:tilt
+    motor_number="2"
+    parent="base_link"
+    color="Blue"
+    x_axis="-1"
+    y_axis="0">
+    <origin xyz="${-(arm_length+arm_offset)} 0 0" rpy="0 0 0" />
+  </xacro:tilt>
+  <!-- Instantiate tilt 3 -->
+  <xacro:tilt
+    motor_number="3"
+    parent="base_link"
+    color="Blue"
+    x_axis="0"
+    y_axis="-1">
+    <origin xyz="0 ${-(arm_length+arm_offset)} 0" rpy="0 0 0" />
+  </xacro:tilt>
+  <xacro:transmisija
+    trans_number="0"
+    joint_name="tilt_0_joint">
+  </xacro:transmisija>
+  <xacro:transmisija
+    trans_number="1"
+    joint_name="tilt_1_joint">
+  </xacro:transmisija>
+  <xacro:transmisija
+    trans_number="2"
+    joint_name="tilt_2_joint">
+  </xacro:transmisija>
+  <xacro:transmisija
+    trans_number="3"
+    joint_name="tilt_3_joint">
+  </xacro:transmisija>
   <!-- Instantiate rotors -->
   <xacro:vertical_rotor
@@ -75,5 +127,5 @@
     motor_constant="${motor_constant}"
     moment_constant="${moment_constant}"
-    parent="base_link"
+    parent="tilt_0"
     mass_rotor="${mass_rotor}"
     radius_rotor="${radius_rotor}"
@@ -84,5 +136,5 @@
     rolling_moment_coefficient="${rolling_moment_coefficient}"
     color="Red">
-    <origin xyz="${arm_length+arm_offset} 0 ${propeler_offset}" rpy="0 0 0" />
+    <origin xyz="0 0 ${propeler_offset}" rpy="0 0 0" />
     <xacro:insert_block name="rotor_inertia" />
   </xacro:vertical_rotor>
@@ -93,5 +145,5 @@
     motor_constant="${motor_constant}"
     moment_constant="${moment_constant}"
-    parent="base_link"
+    parent="tilt_1"
     mass_rotor="${mass_rotor}"
     radius_rotor="${radius_rotor}"
@@ -102,5 +154,5 @@
     rolling_moment_coefficient="${rolling_moment_coefficient}"
     color="Blue">
-    <origin xyz="0 ${arm_length+arm_offset} ${propeler_offset}" rpy="0 0 0" />
+    <origin xyz="0 0 ${propeler_offset}" rpy="0 0 0" />
     <xacro:insert_block name="rotor_inertia" />
   </xacro:vertical_rotor>
@@ -111,5 +163,5 @@
     motor_constant="${motor_constant}"
     moment_constant="${moment_constant}"
-    parent="base_link"
+    parent="tilt_2"
     mass_rotor="${mass_rotor}"
     radius_rotor="${radius_rotor}"
@@ -120,5 +172,5 @@
     rolling_moment_coefficient="${rolling_moment_coefficient}"
     color="Blue">
-    <origin xyz="${-(arm_length+arm_offset)} 0 ${propeler_offset}" rpy="0 0 0" />
+    <origin xyz="0 0 ${propeler_offset}" rpy="0 0 0" />
     <xacro:insert_block name="rotor_inertia" />
   </xacro:vertical_rotor>
@@ -129,5 +181,5 @@
     motor_constant="${motor_constant}"
     moment_constant="${moment_constant}"
-    parent="base_link"
+    parent="tilt_3"
     mass_rotor="${mass_rotor}"
     radius_rotor="${radius_rotor}"
@@ -138,79 +190,7 @@
     rolling_moment_coefficient="${rolling_moment_coefficient}"
     color="Blue">
-    <origin xyz="0 ${-(arm_length+arm_offset)} ${propeler_offset}" rpy="0 0 0" />
-    <xacro:insert_block name="rotor_inertia" />
-  </xacro:vertical_rotor>
-  <!-- Instantiate movable mass 0-->
-  <xacro:movable_mass
-    mass_number="0"
-    parent="base_link"
-    mass="${movable_mass_mass}"
-    dimension="${movable_mass_dimension}"
-    color="Red"
-    x_axis="1"
-    y_axis="0"
-    z_axis="0"
-    orientation="${PI}">
-    <origin xyz="${(arm_length/2+arm_offset)} 0.0 ${movable_mass_offset}" rpy="0 0 0" />
-    <xacro:insert_block name="movable_mass_inertia"/>
-  </xacro:movable_mass>
-  <!-- Instantiate movable mass 1 -->
-  <xacro:movable_mass
-    mass_number="1"
-    parent="base_link"
-    mass="${movable_mass_mass}"
-    dimension="${movable_mass_dimension}"
-    color="Blue"
-    x_axis="0"
-    y_axis="1"
-    z_axis="0"
-    orientation="${PI/2}">
-    <origin xyz="0.0 ${(arm_length/2+arm_offset)} ${movable_mass_offset}" rpy="0 0 0" />
-    <xacro:insert_block name="movable_mass_inertia"/>
-  </xacro:movable_mass>
-  <!-- Instantiate movable mass 2-->
-  <xacro:movable_mass
-    mass_number="2"
-    parent="base_link"
-    mass="${movable_mass_mass}"
-    dimension="${movable_mass_dimension}"
-    color="Blue"
-    x_axis="-1"
-    y_axis="0"
-    z_axis="0"
-    orientation="${PI}">>
-    <origin xyz="${-(arm_length/2+arm_offset)} 0.0 ${movable_mass_offset}" rpy="0 0 0" />
-    <xacro:insert_block name="movable_mass_inertia"/>
-  </xacro:movable_mass>
-  <!-- Instantiate movable mass 3 -->
-  <xacro:movable_mass
-    mass_number="3"
-    parent="base_link"
-    mass="${movable_mass_mass}"
-    dimension="${movable_mass_dimension}"
-    color="Blue"
-    x_axis="0"
-    y_axis="-1"
-    z_axis="0"
-    orientation="${PI/2}">>
-    <origin xyz="0.0 ${-(arm_length/2+arm_offset)} ${movable_mass_offset}" rpy="0 0 0" />
-    <xacro:insert_block name="movable_mass_inertia"/>
-  </xacro:movable_mass>
-  <xacro:transmisija
-    trans_number="0"
-    joint_name="stick_to_movable_mass_0">
-  </xacro:transmisija>
-  <xacro:transmisija
-    trans_number="1"
-    joint_name="stick_to_movable_mass_1">
-  </xacro:transmisija>
-  <xacro:transmisija
-    trans_number="2"
-    joint_name="stick_to_movable_mass_2">
-  </xacro:transmisija>
-  <xacro:transmisija
-    trans_number="3"
-    joint_name="stick_to_movable_mass_3">
-  </xacro:transmisija>
+    <origin xyz="0 0 ${propeler_offset}" rpy="0 0 0" />
+    <xacro:insert_block name="rotor_inertia" />
+  </xacro:vertical_rotor>
   <xacro:property name="land_gear_inertia">
     <inertia

File: morus_description/urdf/multirotor_base.urdf.xacro (robot description, xacro)
@@ -91,4 +91,39 @@
     </link>
     <gazebo reference="movable_mass_${mass_number}">
+      <material>Gazebo/${color}</material>
+    </gazebo>
+  </xacro:macro>
+  <!-- Macro file for tilted props. It defines joint between prop and body, and link which defines actual joint. Stick
+  is defined in other macro file-->
+  <xacro:macro name="tilt" params="parent motor_number x_axis y_axis color *origin">
+    <joint name="tilt_${motor_number}_joint" type="revolute">
+      <xacro:insert_block name="origin"/>
+      <axis xyz="${x_axis} ${y_axis} 0"/>
+      <parent link="${parent}"/>
+      <child link="tilt_${motor_number}"/>
+      <limit lower="-0.785398163" upper="0.785398163" effort="10000" velocity="20"/>
+    </joint>
+    <link name="tilt_${motor_number}">
+      <visual>
+        <geometry>
+          <cylinder length="0.1" radius="0.05" />
+        </geometry>
+      </visual>
+      <collision>
+        <xacro:insert_block name="origin" />
+        <geometry>
+            <cylinder length="0.1" radius="0.05" />
+        </geometry>
+      </collision>
+      <inertial>
+          <xacro:insert_block name="origin" />
+          <mass value="0.1" />
+          <inertia
+            ixx="1.0" ixy="0.0" ixz="0.0"
+            iyy="1.0" iyz="0.0"
+            izz="1.0" />
+      </inertial>
+    </link>
+    <gazebo reference="tilt_${motor_number}">
       <material>Gazebo/${color}</material>
     </gazebo>

Commit message: Adjusted urdf files for new uav collada file. Adjuested model parameters.

File: morus_description/urdf/morus.urdf.xacro (robot description, xacro)
@@ -3,24 +3,25 @@
   <!-- Properties -->
   <xacro:property name="rotor_velocity_slowdown_sim" value="10" />
-  <xacro:property name="mesh_file" value="MORUS_UAV_without_mass.dae" />
+  <xacro:property name="mesh_file" value="morus_uav_final.dae" />
   <xacro:property name="mesh_file_mass" value="MORUS_mass.dae" />
   <xacro:property name="mass" value="30" />  <!-- [kg] -->
-  <xacro:property name="body_width" value="0.3" /> <!-- 0.1 [m] -->
-  <xacro:property name="body_height" value="0.25" /> <!--0.2 [m] -->
+   <xacro:property name="body_width" value="0.35" /> <!-- 0.1 [m] -->
+  <xacro:property name="body_height" value="0.15" /> <!--0.2 [m] -->
   <xacro:property name="mass_rotor" value="0.2" /> <!-- [kg] -->
-  <xacro:property name="arm_length" value="0.515" /> <!-- [m] -->
-  <xacro:property name="arm_offset" value="0.1" /> <!-- [m] -->
-  <xacro:property name="propeler_offset" value="0.325" /> <!-- [m] -->
-  <xacro:property name="rotor_offset_top" value="0.037" /> <!-- [m] -->
+  <xacro:property name="arm_length" value="0.65" /> <!-- [m] -->
+  <xacro:property name="arm_offset" value="0.175" /> <!-- [m] -->
+  <xacro:property name="prop_ver_offset" value="0.15" /> <!-- [m] -->
+  <xacro:property name="prop_long_offset" value="0.07" /> <!-- [m] -->
   <xacro:property name="radius_rotor" value="0.33" /> <!-- [m] -->
   <xacro:property name="motor_constant" value="0.000456874" /> <!-- [kg*m/s^2] -->
-  <xacro:property name="moment_constant" value="0.01" /> <!-- [m] -->
-  <xacro:property name="time_constant" value="0.125" /> <!-- [s] -->s ti
+  <xacro:property name="moment_constant" value="0.025" /> <!-- [m] -->
+  <xacro:property name="time_constant_up" value="0.2" /> <!-- [s] -->
+  <xacro:property name="time_constant_down" value="0.2" /> <!-- [s] -->
   <xacro:property name="max_rot_velocity" value="838" /> <!-- [rad/s] -->
-  <xacro:property name="rotor_drag_coefficient" value="8.06428e-04" />
+  <xacro:property name="rotor_drag_coefficient" value="0.0" /> <!--8.06428e-03-->
   <xacro:property name="rolling_moment_coefficient" value="0.00001" />
   <xacro:property name="movable_mass_mass" value="1" />
   <xacro:property name="movable_mass_dimension" value="0.08" />
-  <xacro:property name="movable_mass_offset" value="0.025" />
+  <xacro:property name="movable_mass_offset" value="0.05" />
   <xacro:property name="imu_mass" value="0.02"/>
   <xacro:property name="imu_size" value="0.01"/>
@@ -30,5 +31,6 @@
   <!-- Property Blocks -->
   <xacro:property name="body_inertia">
-    <inertia ixx="5.5268" ixy="0.0" ixz="0.0" iyy="5.5268" iyz="0.0" izz="6.8854" />
+    <!--inertia ixx="8.66" ixy="0.0" ixz="0.0" iyy="8.66" iyz="0.0" izz="12.0" /!-->
+    <inertia ixx="5.5" ixy="0.0" ixz="0.0" iyy="5.5" iyz="0.0" izz="6.5" />
   </xacro:property>
   <!-- inertia of a single rotor, assuming it is a cuboid. Height=3mm, width=15mm -->
@@ -68,5 +70,5 @@
     <xacro:insert_block name="body_inertia" />
   </xacro:multirotor_base_macro>
-  <!-- Instantiate rotors -->
+ <!-- Instantiate rotors -->
   <xacro:vertical_rotor
     robot_namespace="$(arg name)"
@@ -78,5 +80,6 @@
     mass_rotor="${mass_rotor}"
     radius_rotor="${radius_rotor}"
-    time_constant="${time_constant}"
+    time_constant_up="${time_constant_up}"
+    time_constant_down="${time_constant_down}"
     max_rot_velocity="${max_rot_velocity}"
     motor_number="0"
@@ -84,5 +87,5 @@
     rolling_moment_coefficient="${rolling_moment_coefficient}"
     color="Red">
-    <origin xyz="${arm_length+arm_offset} 0 ${propeler_offset}" rpy="0 0 0" />
+    <origin xyz="${arm_length+prop_long_offset+arm_offset} 0 ${prop_ver_offset}" rpy="0 0 0" />
     <xacro:insert_block name="rotor_inertia" />
   </xacro:vertical_rotor>
@@ -96,5 +99,6 @@
     mass_rotor="${mass_rotor}"
     radius_rotor="${radius_rotor}"
-    time_constant="${time_constant}"
+    time_constant_up="${time_constant_up}"
+    time_constant_down="${time_constant_down}"
     max_rot_velocity="${max_rot_velocity}"
     motor_number="1"
@@ -102,5 +106,5 @@
     rolling_moment_coefficient="${rolling_moment_coefficient}"
     color="Blue">
-    <origin xyz="0 ${arm_length+arm_offset} ${propeler_offset}" rpy="0 0 0" />
+    <origin xyz="0 ${arm_length+prop_long_offset+arm_offset} ${prop_ver_offset}" rpy="0 0 0" />
     <xacro:insert_block name="rotor_inertia" />
   </xacro:vertical_rotor>
@@ -114,5 +118,6 @@
     mass_rotor="${mass_rotor}"
     radius_rotor="${radius_rotor}"
-    time_constant="${time_constant}"
+    time_constant_up="${time_constant_up}"
+    time_constant_down="${time_constant_down}"
     max_rot_velocity="${max_rot_velocity}"
     motor_number="2"
@@ -120,5 +125,5 @@
     rolling_moment_coefficient="${rolling_moment_coefficient}"
     color="Blue">
-    <origin xyz="${-(arm_length+arm_offset)} 0 ${propeler_offset}" rpy="0 0 0" />
+    <origin xyz="${-(arm_length+prop_long_offset+arm_offset)} 0 ${prop_ver_offset}" rpy="0 0 0" />
     <xacro:insert_block name="rotor_inertia" />
   </xacro:vertical_rotor>
@@ -132,5 +137,6 @@
     mass_rotor="${mass_rotor}"
     radius_rotor="${radius_rotor}"
-    time_constant="${time_constant}"
+    time_constant_up="${time_constant_up}"
+    time_constant_down="${time_constant_down}"
     max_rot_velocity="${max_rot_velocity}"
     motor_number="3"
@@ -138,5 +144,5 @@
     rolling_moment_coefficient="${rolling_moment_coefficient}"
     color="Blue">
-    <origin xyz="0 ${-(arm_length+arm_offset)} ${propeler_offset}" rpy="0 0 0" />
+    <origin xyz="0 ${-(arm_length+prop_long_offset+arm_offset)} ${prop_ver_offset}" rpy="0 0 0" />
     <xacro:insert_block name="rotor_inertia" />
   </xacro:vertical_rotor>
@@ -179,5 +185,5 @@
     y_axis="0"
     z_axis="0"
-    orientation="${PI}">>
+    orientation="${PI}">
     <origin xyz="${-(arm_length/2+arm_offset)} 0.0 ${movable_mass_offset}" rpy="0 0 0" />
     <xacro:insert_block name="movable_mass_inertia"/>
@@ -193,5 +199,5 @@
     y_axis="-1"
     z_axis="0"
-    orientation="${PI/2}">>
+    orientation="${PI/2}">
     <origin xyz="0.0 ${-(arm_length/2+arm_offset)} ${movable_mass_offset}" rpy="0 0 0" />
     <xacro:insert_block name="movable_mass_inertia"/>
@@ -224,8 +230,8 @@
       gear_num = "1"
       mass = "1e-6"
-      dim_x = "0.8"
-      dim_y = "0.1"
-      dim_z = "0.05">
-      <origin xyz="0 -0.325 -0.6" rpy="0 0 0" />
+      dim_x = "0.12"
+      dim_y = "0.04"
+      dim_z = "0.0001">
+      <origin xyz="0 -0.7 -0.275" rpy="0 0 0" />
       <xacro:insert_block name="land_gear_inertia"/>
   </xacro:landing_gear>
@@ -234,8 +240,28 @@
       gear_num = "2"
       mass = "1e-6"
-      dim_x = "0.8"
-      dim_y = "0.1"
-      dim_z = "0.05">
-      <origin xyz="0 0.325 -0.6" rpy="0 0 0" />
+      dim_x = "0.12"
+      dim_y = "0.04"
+      dim_z = "0.0001">
+      <origin xyz="0 0.7 -0.275" rpy="0 0 0" />
+      <xacro:insert_block name="land_gear_inertia"/>
+  </xacro:landing_gear>
+  <xacro:landing_gear
+      parent="base_link"
+      gear_num = "3"
+      mass = "1e-6"
+      dim_x = "0.12"
+      dim_y = "0.04"
+      dim_z = "0.0001">
+      <origin xyz="-0.7 0 -0.275" rpy="0 0 1.57" />
+      <xacro:insert_block name="land_gear_inertia"/>
+  </xacro:landing_gear>
+  <xacro:landing_gear
+      parent="base_link"
+      gear_num = "4"
+      mass = "1e-6"
+      dim_x = "0.12"
+      dim_y = "0.04"
+      dim_z = "0.0001">
+      <origin xyz="0.7 0.0 -0.275" rpy="0 0 1.57" />
       <xacro:insert_block name="land_gear_inertia"/>
   </xacro:landing_gear>

File: morus_description/urdf/multirotor_base.urdf.xacro (robot description, xacro)
@@ -17,8 +17,8 @@
       </inertial>
       <visual>
-        <origin xyz="0 0 0.125" rpy="0 0 0" />
+        <origin xyz="0 0 -0.65" rpy="0 0 0" />
         <geometry>
           <mesh filename="package://morus_description/meshes/${mesh_file}"
-            scale="1 1 1" />
+            scale="0.001 0.001 0.001" />
           <!--box size="${body_width} ${body_width} ${body_height}"/--> <!-- [m] [m] [m] -->
         </geometry>
@@ -71,5 +71,5 @@
       <visual>
         <!--origin rpy="0 0 ${orientation}" xyz="0 0 ${0*movable_mass_dimension/2}"/-->
-        <origin rpy="0 0 ${orientation}" xyz="0 0 0"/>
+        <origin rpy="0 0 ${orientation}" xyz="0 0 -0.05"/>
         <geometry>
           <!--mesh filename="package://morus_description/meshes/${mesh_file_mass}"
@@ -96,5 +96,5 @@
   <!-- Rotor joint and link -->
   <xacro:macro name="vertical_rotor"
-    params="robot_namespace suffix direction motor_constant moment_constant parent mass_rotor radius_rotor time_constant max_rot_velocity motor_number rotor_drag_coefficient rolling_moment_coefficient color *origin *inertia">
+    params="robot_namespace suffix direction motor_constant moment_constant parent mass_rotor radius_rotor time_constant_up time_constant_down max_rot_velocity motor_number rotor_drag_coefficient rolling_moment_coefficient color *origin *inertia">
     <joint name="rotor_${motor_number}_joint" type="continuous">
       <xacro:insert_block name="origin" />
@@ -132,5 +132,6 @@
         <linkName>rotor_${motor_number}</linkName>
         <turningDirection>${direction}</turningDirection>
-        <timeConstant>${time_constant}</timeConstant>
+        <timeConstantUp>${time_constant_up}</timeConstantUp>
+        <timeConstantDown>${time_constant_down}</timeConstantDown>
         <maxRotVelocity>${max_rot_velocity}</maxRotVelocity>
         <motorConstant>${motor_constant}</motorConstant>
