Commit message: Revert "finished control flap model"
This reverts commit 9efafe536a9817014320bebeedb35ea5065b1c76.

File: morus_description/urdf/morus.urdf.xacro (robot description, xacro)
@@ -20,27 +20,4 @@
   <xacro:property name="rotor_drag_coefficient" value="8.06428e-04" />
   <xacro:property name="rolling_moment_coefficient" value="0.00001" />
-  <!--wing properties -->
-  <xacro:property name="wing_mass" value="0.001"/> <!-- [kg] -->
-  <xacro:property name="wing_x" value="0.01"/> <!-- [m] -->
-  <xacro:property name="wing_y" value="0.66"/> <!-- [m] -->
-  <xacro:property name="wing_z" value="0.1"/> <!-- [m] -->
-  <xacro:property name="arm_height" value="0.1" /> <!-- [m] added arm_height for no wing-rotor interaction -->
-  <xacro:property name="area_control_flap" value="0.066"/> <!-- [m^2] -->
-  <xacro:property name="area_antitorque_flap" value="0.066"/> <!-- [m^2] -->
-  <!--realistic rotor properties -->
-  <xacro:property name="fluid_density" value="1.2041" />  <!-- air -->
-  <xacro:property name="distance_antitorque_flap" value="0.08" /> <!-- [m] distance from centre of gravity of rotor, force*distance=moment-->
-  <xacro:property name="distance_control_flap" value="0.1" /> <!-- [m] -->
-  <xacro:property name="thrust_coefficient" value="0.000456874" />  <!-- motor_constant Kf-->
-  <xacro:property name="torque_coefficient" value="0.01" /> <!-- moment_constant Kt-->
-  <xacro:property name="slip_velocity_coefficient" value="2.7e-02" /> <!-- Kv -->
-  <xacro:property name="lift_coefficient_control_flap" value="8.5e-02" />  <!-- Clc -->
-  <xacro:property name="drag_coefficient_control_flap" value="1.3e-01" />  <!-- Cdc -->
-  <xacro:property name="lift_coefficient_antitorque_flap" value="3.4e-02" />  <!-- Cla -->
-  <xacro:property name="drag_coefficient_antitorque_flap" value="1.3e-01" />  <!-- Cda -->
-  <xacro:property name="lift_coefficient_control_flap_at0" value="0" />  <!-- Clc0 not used in the formulas -->
-  <xacro:property name="drag_coefficient_control_flap_at0" value="7.47e-03" />  <!-- Cdc0 -->
-  <xacro:property name="lift_coefficient_antitorque_flap_at0" value="1.358e-01" />  <!-- Cla0 -->
-  <xacro:property name="drag_coefficient_antitorque_flap_at0" value="3.23e-03" />  <!-- Cda0 -->
   <xacro:property name="movable_mass_mass" value="1" />
   <xacro:property name="movable_mass_dimension" value="0.08" />
@@ -51,5 +28,4 @@
   <xacro:property name="cos45" value="0.7071" />
   <xacro:property name="PI" value="3.14" />
-  <xacro:property name="PIhalf" value="1.5707" />
   <!-- Property Blocks -->
   <xacro:property name="body_inertia">
@@ -80,12 +56,4 @@
     ixy="0.0" ixz="0.0"  iyz="0.0" /> <!-- [kg*m^2] [kg*m^2] [kg*m^2] [kg*m^2] [kg*m^2] [kg*m^2] -->
   </xacro:property>
-  <!-- wing inertia -->
-  <xacro:property name="wing_inertia">
-    <inertia
-    ixx="${(wing_mass * wing_x * wing_x)/6}"
-    iyy="${(wing_mass * wing_y * wing_y)/6}"
-    izz="${(wing_mass * wing_z * wing_z)/6}"
-    ixy="0.0" ixz="0.0"  iyz="0.0" /> <!-- [kg*m^2] [kg*m^2] [kg*m^2] [kg*m^2] [kg*m^2] [kg*m^2] -->
-  </xacro:property>
   <!-- Included URDF Files -->
   <xacro:include filename="$(find morus_description)/urdf/multirotor_base.urdf.xacro" />
@@ -100,66 +68,5 @@
     <xacro:insert_block name="body_inertia" />
   </xacro:multirotor_base_macro>
-  <!-- Instantiate wing 0 -->
-  <xacro:wing
-    robot_namespace="$(arg name)"
-    parent="base_link"
-    wing_number="0"
-    mass="${wing_mass}"
-    wing_x="${wing_x}"
-    wing_y="${wing_y}"
-    wing_z="${wing_z}"
-    x_axis="0"
-    y_axis="1"
-    color="Red">
-    <origin xyz="${arm_length+arm_offset} 0 ${-arm_height}" rpy="0 0 0" />
-    <xacro:insert_block name="wing_inertia"/>
-  </xacro:wing>
-  <!-- Instantiate wing 1-->
-  <xacro:wing
-    robot_namespace="$(arg name)"
-    parent="base_link"
-    wing_number="1"
-    mass="${wing_mass}"
-    wing_x="${wing_x}"
-    wing_y="${wing_y}"
-    wing_z="${wing_z}"
-    x_axis="0"
-    y_axis="1"
-    color="Blue">
-    <origin xyz="0 ${arm_length+arm_offset} ${-arm_height}" rpy="0 0 ${PIhalf}" />
-    <xacro:insert_block name="wing_inertia"/>
-  </xacro:wing>
-  <!-- same x_axis and y_axis values as wing 0 because rpy flips the coordinate system by PIhalf-->
-  <!-- Instantiate wing 2-->
-  <xacro:wing
-    robot_namespace="$(arg name)"
-    parent="base_link"
-    wing_number="2"
-    mass="${wing_mass}"
-    wing_x="${wing_x}"
-    wing_y="${wing_y}"
-    wing_z="${wing_z}"
-    x_axis="0"
-    y_axis="1"
-    color="Blue">
-    <origin xyz="${-(arm_length+arm_offset)} 0 ${-arm_height}" rpy="0 0 0" />
-    <xacro:insert_block name="wing_inertia"/>
-  </xacro:wing>
-  <!-- Instantiate wing 3-->
-  <xacro:wing
-    robot_namespace="$(arg name)"
-    parent="base_link"
-    wing_number="3"
-    mass="${wing_mass}"
-    wing_x="${wing_x}"
-    wing_y="${wing_y}"
-    wing_z="${wing_z}"
-    x_axis="0"
-    y_axis="1"
-    color="Blue">
-    <origin xyz="0 ${-(arm_length+arm_offset)} ${-arm_height}" rpy="0 0 ${PIhalf}" />
-    <xacro:insert_block name="wing_inertia"/>
-  </xacro:wing>
-  <!-- Instantiate tilt 0
+  <!-- Instantiate tilt 0-->
   <xacro:tilt
     motor_number="0"
@@ -169,6 +76,6 @@
     y_axis="0">
     <origin xyz="${arm_length+arm_offset} 0 0" rpy="0 0 0" />
-  </xacro:tilt>-->
-  <!-- Instantiate tilt 1
+  </xacro:tilt>
+  <!-- Instantiate tilt 1 -->
   <xacro:tilt
     motor_number="1"
@@ -178,6 +85,6 @@
     y_axis="1">
     <origin xyz="0 ${arm_length+arm_offset} 0" rpy="0 0 0" />
-  </xacro:tilt>-->
-  <!-- Instantiate tilt 2
+  </xacro:tilt>
+  <!-- Instantiate tilt 2-->
   <xacro:tilt
     motor_number="2"
@@ -187,6 +94,6 @@
     y_axis="0">
     <origin xyz="${-(arm_length+arm_offset)} 0 0" rpy="0 0 0" />
-  </xacro:tilt>-->
-  <!-- Instantiate tilt 3
+  </xacro:tilt>
+  <!-- Instantiate tilt 3 -->
   <xacro:tilt
     motor_number="3"
@@ -196,22 +103,22 @@
     y_axis="-1">
     <origin xyz="0 ${-(arm_length+arm_offset)} 0" rpy="0 0 0" />
-  </xacro:tilt>-->
+  </xacro:tilt>
   <xacro:transmisija
     trans_number="0"
-    joint_name="wing_0_joint"> <!-- tilt_0_joint -->
+    joint_name="tilt_0_joint">
   </xacro:transmisija>
   <xacro:transmisija
     trans_number="1"
-    joint_name="wing_1_joint">
+    joint_name="tilt_1_joint">
   </xacro:transmisija>
   <xacro:transmisija
     trans_number="2"
-    joint_name="wing_2_joint">
+    joint_name="tilt_2_joint">
   </xacro:transmisija>
   <xacro:transmisija
     trans_number="3"
-    joint_name="wing_3_joint">
-  </xacro:transmisija>
-  <!-- Instantiate rotors -->   <!-- tilt_0-->
+    joint_name="tilt_3_joint">
+  </xacro:transmisija>
+  <!-- Instantiate rotors -->
   <xacro:vertical_rotor
     robot_namespace="$(arg name)"
@@ -220,21 +127,5 @@
     motor_constant="${motor_constant}"
     moment_constant="${moment_constant}"
-    area_control_flap="${area_control_flap}"
-    area_antitorque_flap="${area_antitorque_flap}"
-    fluid_density ="${fluid_density}"
-    distance_control_flap="${distance_control_flap}"
-    distance_antitorque_flap="${distance_antitorque_flap}"
-    thrust_coefficient="${thrust_coefficient}"
-    torque_coefficient="${torque_coefficient}"
-    slip_velocity_coefficient="${slip_velocity_coefficient}"
-    lift_coefficient_control_flap="${lift_coefficient_control_flap}"
-    drag_coefficient_control_flap="${drag_coefficient_control_flap}"
-    lift_coefficient_antitorque_flap="${lift_coefficient_antitorque_flap}"
-    drag_coefficient_antitorque_flap="${drag_coefficient_antitorque_flap}"
-    lift_coefficient_control_flap_at0="${lift_coefficient_control_flap_at0}"
-    drag_coefficient_control_flap_at0="${drag_coefficient_control_flap_at0}"
-    lift_coefficient_antitorque_flap_at0="${lift_coefficient_antitorque_flap_at0}"
-    drag_coefficient_antitorque_flap_at0="${drag_coefficient_antitorque_flap_at0}"
-    parent="base_link"
+    parent="tilt_0"
     mass_rotor="${mass_rotor}"
     radius_rotor="${radius_rotor}"
@@ -245,5 +136,5 @@
     rolling_moment_coefficient="${rolling_moment_coefficient}"
     color="Red">
-    <origin xyz="${arm_length+arm_offset} 0 ${propeler_offset}" rpy="0 0 0" />
+    <origin xyz="0 0 ${propeler_offset}" rpy="0 0 0" />
     <xacro:insert_block name="rotor_inertia" />
   </xacro:vertical_rotor>
@@ -254,21 +145,5 @@
     motor_constant="${motor_constant}"
     moment_constant="${moment_constant}"
-    area_control_flap="${area_control_flap}"
-    area_antitorque_flap="${area_antitorque_flap}"
-    fluid_density ="${fluid_density}"
-    distance_control_flap="${distance_control_flap}"
-    distance_antitorque_flap="${distance_antitorque_flap}"
-    thrust_coefficient="${thrust_coefficient}"
-    torque_coefficient="${torque_coefficient}"
-    slip_velocity_coefficient="${slip_velocity_coefficient}"
-    lift_coefficient_control_flap="${lift_coefficient_control_flap}"
-    drag_coefficient_control_flap="${drag_coefficient_control_flap}"
-    lift_coefficient_antitorque_flap="${lift_coefficient_antitorque_flap}"
-    drag_coefficient_antitorque_flap="${drag_coefficient_antitorque_flap}"
-    lift_coefficient_control_flap_at0="${lift_coefficient_control_flap_at0}"
-    drag_coefficient_control_flap_at0="${drag_coefficient_control_flap_at0}"
-    lift_coefficient_antitorque_flap_at0="${lift_coefficient_antitorque_flap_at0}"
-    drag_coefficient_antitorque_flap_at0="${drag_coefficient_antitorque_flap_at0}"
-    parent="base_link"
+    parent="tilt_1"
     mass_rotor="${mass_rotor}"
     radius_rotor="${radius_rotor}"
@@ -279,5 +154,5 @@
     rolling_moment_coefficient="${rolling_moment_coefficient}"
     color="Blue">
-    <origin xyz="0 ${arm_length+arm_offset} ${propeler_offset}" rpy="0 0 0" />
+    <origin xyz="0 0 ${propeler_offset}" rpy="0 0 0" />
     <xacro:insert_block name="rotor_inertia" />
   </xacro:vertical_rotor>
@@ -288,21 +163,5 @@
     motor_constant="${motor_constant}"
     moment_constant="${moment_constant}"
-    area_control_flap="${area_control_flap}"
-    area_antitorque_flap="${area_antitorque_flap}"
-    fluid_density ="${fluid_density}"
-    distance_control_flap="${distance_control_flap}"
-    distance_antitorque_flap="${distance_antitorque_flap}"
-    thrust_coefficient="${thrust_coefficient}"
-    torque_coefficient="${torque_coefficient}"
-    slip_velocity_coefficient="${slip_velocity_coefficient}"
-    lift_coefficient_control_flap="${lift_coefficient_control_flap}"
-    drag_coefficient_control_flap="${drag_coefficient_control_flap}"
-    lift_coefficient_antitorque_flap="${lift_coefficient_antitorque_flap}"
-    drag_coefficient_antitorque_flap="${drag_coefficient_antitorque_flap}"
-    lift_coefficient_control_flap_at0="${lift_coefficient_control_flap_at0}"
-    drag_coefficient_control_flap_at0="${drag_coefficient_control_flap_at0}"
-    lift_coefficient_antitorque_flap_at0="${lift_coefficient_antitorque_flap_at0}"
-    drag_coefficient_antitorque_flap_at0="${drag_coefficient_antitorque_flap_at0}"
-    parent="base_link"
+    parent="tilt_2"
     mass_rotor="${mass_rotor}"
     radius_rotor="${radius_rotor}"
@@ -313,5 +172,5 @@
     rolling_moment_coefficient="${rolling_moment_coefficient}"
     color="Blue">
-    <origin xyz="${-(arm_length+arm_offset)} 0 ${propeler_offset}" rpy="0 0 0" />
+    <origin xyz="0 0 ${propeler_offset}" rpy="0 0 0" />
     <xacro:insert_block name="rotor_inertia" />
   </xacro:vertical_rotor>
@@ -322,21 +181,5 @@
     motor_constant="${motor_constant}"
     moment_constant="${moment_constant}"
-    area_control_flap="${area_control_flap}"
-    area_antitorque_flap="${area_antitorque_flap}"
-    fluid_density ="${fluid_density}"
-    distance_control_flap="${distance_control_flap}"
-    distance_antitorque_flap="${distance_antitorque_flap}"
-    thrust_coefficient="${thrust_coefficient}"
-    torque_coefficient="${torque_coefficient}"
-    slip_velocity_coefficient="${slip_velocity_coefficient}"
-    lift_coefficient_control_flap="${lift_coefficient_control_flap}"
-    drag_coefficient_control_flap="${drag_coefficient_control_flap}"
-    lift_coefficient_antitorque_flap="${lift_coefficient_antitorque_flap}"
-    drag_coefficient_antitorque_flap="${drag_coefficient_antitorque_flap}"
-    lift_coefficient_control_flap_at0="${lift_coefficient_control_flap_at0}"
-    drag_coefficient_control_flap_at0="${drag_coefficient_control_flap_at0}"
-    lift_coefficient_antitorque_flap_at0="${lift_coefficient_antitorque_flap_at0}"
-    drag_coefficient_antitorque_flap_at0="${drag_coefficient_antitorque_flap_at0}"
-    parent="base_link"
+    parent="tilt_3"
     mass_rotor="${mass_rotor}"
     radius_rotor="${radius_rotor}"
@@ -347,5 +190,5 @@
     rolling_moment_coefficient="${rolling_moment_coefficient}"
     color="Blue">
-    <origin xyz="0 ${-(arm_length+arm_offset)} ${propeler_offset}" rpy="0 0 0" />
+    <origin xyz="0 0 ${propeler_offset}" rpy="0 0 0" />
     <xacro:insert_block name="rotor_inertia" />
   </xacro:vertical_rotor>

File: morus_description/urdf/multirotor_base.urdf.xacro (robot description, xacro)
@@ -95,5 +95,5 @@
   </xacro:macro>
   <!-- Macro file for tilted props. It defines joint between prop and body, and link which defines actual joint. Stick
-  is defined in other macro file
+  is defined in other macro file-->
   <xacro:macro name="tilt" params="parent motor_number x_axis y_axis color *origin">
     <joint name="tilt_${motor_number}_joint" type="revolute">
@@ -128,59 +128,8 @@
       <material>Gazebo/${color}</material>
     </gazebo>
-  </xacro:macro>  -->
-  <!-- Macro file for the wing. It defines joint between base and wing.-->
-  <xacro:macro name="wing"
-     params="robot_namespace parent wing_number mass wing_x wing_y wing_z x_axis y_axis color *origin *inertia">
-    <joint name="wing_${wing_number}_joint" type="revolute">
-    <xacro:insert_block name="origin" />
-      <axis xyz="${x_axis} ${y_axis} 0"/>
-      <parent link="${parent}"/>
-      <child link="wing_${wing_number}"/>
-      <limit lower="-0.261799388" upper="0.261799388" effort="10000" velocity="10"/>
-    </joint>
-    <link name="wing_${wing_number}">
-      <visual>
-        <origin rpy="0 0 0" xyz="0 0 0"/>
-        <geometry>
-          <box size="${1*wing_x} ${1*wing_y} ${1*wing_z}"/>
-        </geometry>
-      </visual>
-      <collision>
-        <origin rpy="0 0 0" xyz="0 0 0"/>
-        <geometry>
-          <box size="${wing_x} ${wing_y} ${wing_z}"/>
-        </geometry>
-      </collision>
-      <inertial>
-        <origin rpy="0 0 0" xyz="0 0 0"/>
-        <mass value="${wing_mass}"/>
-        <xacro:insert_block name="inertia"/>
-      </inertial>
-    </link>
-    <!--gazebo>
-      <plugin name="lifting_surface_${wing_number}" filename="libLiftDragPlugin.so">
-        <a0>0</a0>
-        <alpha_stall>0.3368</alpha_stall>
-        <cla>5.418</cla>
-        <cla_stall>-2.1419</cla_stall>
-        <cda>0.0</cda>
-        <cda_stall>0.0</cda_stall>
-        <cma>0.0</cma>
-        <cma_stall>0.0</cma_stall>
-        <area>3</area>
-        <fluid_density>1.2041</fluid_density>
-        <forward>-1 0 0</forward>
-        <upward>0 -1 0</upward>
-        <cp>0 0 1</cp>
-        <control_joint_name>wing_${wing_number}_joint</control_joint_name>
-      </plugin>
-    </gazebo-->
-    <gazebo reference="wing_${wing_number}">
-      <material>Gazebo/${color}</material>
-    </gazebo>
-</xacro:macro>
+  </xacro:macro>
   <!-- Rotor joint and link -->
   <xacro:macro name="vertical_rotor"
-    params="robot_namespace suffix direction motor_constant moment_constant area_control_flap area_antitorque_flap fluid_density distance_control_flap distance_antitorque_flap thrust_coefficient torque_coefficient slip_velocity_coefficient lift_coefficient_control_flap drag_coefficient_control_flap lift_coefficient_antitorque_flap drag_coefficient_antitorque_flap lift_coefficient_control_flap_at0 drag_coefficient_control_flap_at0 lift_coefficient_antitorque_flap_at0 drag_coefficient_antitorque_flap_at0 parent mass_rotor radius_rotor time_constant max_rot_velocity motor_number rotor_drag_coefficient rolling_moment_coefficient color *origin *inertia">
+    params="robot_namespace suffix direction motor_constant moment_constant parent mass_rotor radius_rotor time_constant max_rot_velocity motor_number rotor_drag_coefficient rolling_moment_coefficient color *origin *inertia">
     <joint name="rotor_${motor_number}_joint" type="continuous">
       <xacro:insert_block name="origin" />
@@ -214,5 +163,5 @@
     </link>
     <gazebo>
-      <plugin name="${suffix}_motor_model" filename="libmorus_gazebo_ductedfan_motor_model.so">
+      <plugin name="${suffix}_motor_model" filename="librotors_gazebo_motor_model.so">
         <jointName>rotor_${motor_number}_joint</jointName>
         <linkName>rotor_${motor_number}</linkName>
@@ -228,23 +177,4 @@
         <motorVelocityTopic>${robot_namespace}/motor_vel/${motor_number}</motorVelocityTopic>
         <rotorVelocitySlowdownSim>${rotor_velocity_slowdown_sim}</rotorVelocitySlowdownSim>
-        <angleControlFlapRefSubTopic>morus/angle_wing_${motor_number}_ref_value</angleControlFlapRefSubTopic>
-        <angleControlFlapCommandPubTopic>morus/angle_wing_${motor_number}_controller/command</angleControlFlapCommandPubTopic>
-        <angleControlFlapValueSubTopic>morus/angle_wing_${motor_number}_controller/state</angleControlFlapValueSubTopic>
-        <fluidDensity>${fluid_density}</fluidDensity>
-        <areaControlFlap>${area_control_flap}</areaControlFlap>
-        <areaAntitorqueFlap>${area_antitorque_flap}</areaAntitorqueFlap>
-        <distanceControlFlap>${distance_control_flap}</distanceControlFlap>
-        <distanceAntitorqueFlap>${distance_antitorque_flap}</distanceAntitorqueFlap>
-        <thrustCoefficient>${thrust_coefficient}</thrustCoefficient>
-        <torqueCoefficient>${torque_coefficient}</torqueCoefficient>
-        <slipVelocityCoefficient>${slip_velocity_coefficient}</slipVelocityCoefficient>
-        <liftCoefficientControlFlap>${lift_coefficient_control_flap}</liftCoefficientControlFlap>
-        <dragCoefficientControlFlap>${drag_coefficient_control_flap}</dragCoefficientControlFlap>
-        <liftCoefficientAntitorqueFlap>${lift_coefficient_antitorque_flap}</liftCoefficientAntitorqueFlap>
-        <dragCoefficientAntitorqueFlap>${drag_coefficient_antitorque_flap}</dragCoefficientAntitorqueFlap>
-        <liftCoefficientControlFlapAt0>${lift_coefficient_control_flap_at0}</liftCoefficientControlFlapAt0>
-        <dragCoefficientControlFlapAt0>${drag_coefficient_control_flap_at0}</dragCoefficientControlFlapAt0>
-        <liftCoefficientAntitorqueFlapAt0>${lift_coefficient_antitorque_flap_at0}</liftCoefficientAntitorqueFlapAt0>
-        <dragCoefficientAntitorqueFlapAt0>${drag_coefficient_antitorque_flap_at0}</dragCoefficientAntitorqueFlapAt0>
       </plugin>
     </gazebo>

Commit message: Add camera to morus

File: morus_description/urdf/morus.urdf.xacro (robot description, xacro)
@@ -240,3 +240,20 @@
       <xacro:insert_block name="land_gear_inertia"/>
   </xacro:landing_gear>
+  <!-- Camera properties -->
+  <xacro:property name="camera_link" value="0.05" />
+  <xacro:property name="camera_inertia">
+    <inertia
+    ixx="1e-6"
+    iyy="1e-6"
+    izz="1e-6"
+    ixy="0.0" ixz="0.0" iyz="0.0" />
+  </xacro:property>
+  <xacro:property name="camera_mass" value="1e-5"/>
+  <xacro:cam
+    camera_link="${camera_link}"
+    camera_mass="${camera_mass}"
+    parent="base_link">
+    <origin xyz="0 0 0.5" rpy="0 0 0"/>
+    <xacro:insert_block name="camera_inertia"/>
+  </xacro:cam>
 </robot>

File: morus_description/urdf/multirotor_base.urdf.xacro (robot description, xacro)
@@ -255,3 +255,77 @@
     </gazebo>
   </xacro:macro>
+    <!-- Camera macro. Adds a box representing a camera below the UAV
+  @param camera_link Length of the camera box
+  @param camera_mass Mass of the camera
+  @param parent Parent link on which the camera will be fixed
+  @param *origin Block argument defining the origin of the camera with
+  reference to the parent link.
+  @param *inertia Block argument defining camera inertia.
+  -->
+  <xacro:macro name="cam" params="camera_link camera_mass parent *origin *inertia">
+    <!-- Camera link -->
+    <link name="camera_box">
+      <!--collision>
+        <origin xyz="0 0 0" rpy="0 0 0"/>
+        <geometry>
+          <box size="${camera_link} ${camera_link} ${camera_link}"/>
+        </geometry>
+      </collision-->
+      <visual>
+        <origin xyz="0 0 0" rpy="0 0 0"/>
+        <geometry>
+          <box size="${camera_link} ${camera_link} ${camera_link}"/>
+        </geometry>
+        <material name="red"/>
+      </visual>
+      <inertial>
+        <mass value="${camera_mass}" />
+        <origin xyz="0 0 0" rpy="0 0 0"/>
+        <xacro:insert_block name="inertia"/>
+      </inertial>
+    </link>
+    <!-- Camera joint with reference to the parent link -->
+    <joint name="camera_joint" type="fixed">
+      <xacro:insert_block name="origin"/>
+      <parent link="${parent}"/>
+      <child link="camera_box"/>
+    </joint>
+    <!-- camera -->
+    <gazebo reference="camera_box">
+      <sensor type="camera" name="camera1">
+        <update_rate>30.0</update_rate>
+        <camera name="head">
+          <horizontal_fov>1.3962634</horizontal_fov>
+          <image>
+            <width>800</width>
+            <height>800</height>
+            <format>R8G8B8</format>
+          </image>
+          <clip>
+            <near>0.02</near>
+            <far>300</far>
+          </clip>
+          <noise>
+            <type>gaussian</type>
+            <mean>0.0</mean>
+            <stddev>0.007</stddev>
+          </noise>
+        </camera>
+        <plugin name="camera_controller" filename="libgazebo_ros_camera.so">
+          <alwaysOn>true</alwaysOn>
+          <updateRate>0.0</updateRate>
+          <cameraName>morus/camera1</cameraName>
+          <imageTopicName>image_raw</imageTopicName>
+          <cameraInfoTopicName>camera_info</cameraInfoTopicName>
+          <frameName>camera_box</frameName>
+          <hackBaseline>0.07</hackBaseline>
+          <distortionK1>0.0</distortionK1>
+          <distortionK2>0.0</distortionK2>
+          <distortionK3>0.0</distortionK3>
+          <distortionT1>0.0</distortionT1>
+          <distortionT2>0.0</distortionT2>
+        </plugin>
+      </sensor>
+    </gazebo>
+  </xacro:macro>
 </robot>
