Commit message: Change camera configuration

File: morus_description/urdf/morus.urdf.xacro (robot description, xacro)
@@ -254,5 +254,5 @@
     camera_mass="${camera_mass}"
     parent="base_link">
-    <origin xyz="0 0 0.5" rpy="0 0 0"/>
+    <origin xyz="-0.5 0 0.5" rpy="0 0 0"/>
     <xacro:insert_block name="camera_inertia"/>
   </xacro:cam>

File: morus_description/urdf/multirotor_base.urdf.xacro (robot description, xacro)
@@ -296,5 +296,5 @@
         <update_rate>30.0</update_rate>
         <camera name="head">
-          <horizontal_fov>1.3962634</horizontal_fov>
+          <horizontal_fov>1.5</horizontal_fov>
           <image>
             <width>800</width>
@@ -309,5 +309,5 @@
             <type>gaussian</type>
             <mean>0.0</mean>
-            <stddev>0.007</stddev>
+            <stddev>0.01</stddev>
           </noise>
         </camera>

Commit message: Config fixes

File: morus_description/urdf/morus.urdf.xacro (robot description, xacro)
@@ -254,5 +254,5 @@
     camera_mass="${camera_mass}"
     parent="base_link">
-    <origin xyz="-0.5 0 0.5" rpy="0 0 0"/>
+    <origin xyz="-0.75 0 1.5" rpy="0 0.3 0"/>
     <xacro:insert_block name="camera_inertia"/>
   </xacro:cam>
